File: printhead-pcb/pwr.kicad_sch (KiCad schematic)
At the start: 10 parts, among them U3 AP7361C-33E

Commit message: circuit finished?
Parts:
- removed C7: 10µF, symbol Device:C_Polarized
- removed C8: 0.22µF, symbol Device:C
- removed C9: 0.1µF, symbol Device:C
- removed L2: L, symbol Device:L
- removed U3: AP7361C-33E, Package_TO_SOT_SMD:SOT-223-3_TabPin2, symbol Regulator_Linear:AP7361C-33E
- added L1: L, Inductor_SMD:L_0402_1005Metric, symbol Device:L
- C1: renamed from C10; footprint (none) -> Capacitor_SMD:C_0402_1005Metric
- C2: renamed from C11; footprint (none) -> Capacitor_SMD:C_0402_1005Metric
- C3: renamed from C12; footprint (none) -> Capacitor_SMD:C_0402_1005Metric
- D1: renamed from D2; value LED -> GREEN; footprint (none) -> LED_SMD:LED_0805_2012Metric
- R19: renamed from R5; footprint (none) -> Resistor_SMD:R_0402_1005Metric
Connections:
- net +3V3: now also L1.1; no longer C1.1, C2.1, C3.1
- new net: C1.1, C2.1, C3.1, L1.2
Other:
- moved on the sheet: D1, R19
