File: printhead-pcb/printhead-pcb.kicad_pcb (KiCad board)
At the start: 2 copper layers, 35 x 35 mm, 30 parts, among them J1 Power, J13 Steckverbinder_Male_1, J3 DATA, U1 PCA9615DP, U6 AP7361C-33E

Commit message: finished module one design
Parts:
- moved R1 22.6 mm to (125.8, 126.0), turned to -90 degrees
- moved D1 19.3 mm to (122.1, 126.0), turned to 180 degrees
- moved J3 15.6 mm to (129.5, 113.7), turned to 0 degrees
- moved C2 15.1 mm to (124.2, 130.8), turned to 0 degrees
- moved R9 13.8 mm to (126.0, 112.2), turned to 90 degrees
- moved R4 11.6 mm to (122.5, 112.7), turned to 180 degrees
- moved R3 11.4 mm to (118.5, 112.8), turned to 0 degrees
- moved R8 10.9 mm to (126.0, 115.0), turned to 90 degrees
- moved R7 9.39 mm to (122.5, 114.5), turned to 180 degrees
- moved R2 9.18 mm to (118.5, 114.5), turned to 0 degrees
- moved R6 8.12 mm to (126.0, 122.8), turned to -90 degrees
- moved R5 7.87 mm to (126.0, 120.0), turned to -90 degrees
- moved C13 6.04 mm to (114.0, 113.0), turned to 0 degrees
- moved U1 4.46 mm to (120.5, 117.5), turned to 0 degrees
- moved JP1 2.64 mm to (114.0, 116.0), turned to 90 degrees
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Routing:
- net +5V: track 87.5 -> 78.1 mm
- net GND: track 216.8 -> 223.2 mm
- net +3V3: track 17.3 -> 12.8 mm
- net DSCLM: track 8.36 -> 11.9 mm
- net DSDAM: track 8.94 -> 12.4 mm
- net Net-(J1-Pin_3): track 3.74 -> 5.85 mm
- net SCL: track 23.6 -> 22.5 mm
- net SDA: track 20.4 -> 19.3 mm
- net Net-(J1-Pin_1): track 3.75 -> 4.85 mm
- net DSCLP: track 13.4 -> 14.4 mm

Commit message: prepared second module for tomorrow
Parts:
- added C10: 0.1µF, Capacitor_SMD:C_0402_1005Metric, F.Cu at (94.5, 35.9)
- added C11: 0.1µF, Capacitor_SMD:C_0402_1005Metric, F.Cu at (94.5, 37.8)
- added C7: 0.1µF, Capacitor_SMD:C_0402_1005Metric, F.Cu at (94.5, 30.0)
- added C8: 0.1µF, Capacitor_SMD:C_0402_1005Metric, F.Cu at (94.5, 31.9)
- added C9: 0.1µF, Capacitor_SMD:C_0402_1005Metric, F.Cu at (94.5, 33.9)
- added D2: BLUE, LED_SMD:LED_0805_2012Metric, F.Cu at (92.4, 45.1)
- added D3: YELLOW, LED_SMD:LED_0805_2012Metric, F.Cu at (73.5, 67.9)
- added D4: YELLOW, LED_SMD:LED_0805_2012Metric, F.Cu at (73.5, 70.9)
- added H5: MountingHole_Pad, MountingHole:MountingHole_2.2mm_M2_Pad_TopBottom, F.Cu at (153.0, 103.0)
- added H6: MountingHole_Pad, MountingHole:MountingHole_2.2mm_M2_Pad_TopBottom, F.Cu at (182.0, 132.0)
- added H7: MountingHole_Pad, MountingHole:MountingHole_2.2mm_M2_Pad_TopBottom, F.Cu at (182.0, 103.0)
- added H8: MountingHole_Pad, MountingHole:MountingHole_2.2mm_M2_Pad_TopBottom, F.Cu at (153.0, 132.0)
- added J10: T2, Connector_PinHeader_2.54mm:PinHeader_1x02_P2.54mm_Horizontal, F.Cu at (79.0, 45.7)
- added J11: T3, Connector_PinHeader_2.54mm:PinHeader_1x02_P2.54mm_Horizontal, F.Cu at (79.0, 52.9)
- added J12: Breakout_Board_ADXL345, Connector_PinHeader_2.54mm:PinHeader_1x04_P2.54mm_Horizontal, F.Cu at (58.2, 62.1)
- added J2: Fan_12/5V_Regelung, Connector_PinHeader_2.54mm:PinHeader_1x03_P2.54mm_Horizontal, F.Cu at (63.6, 31.3)
- added J4: FAN0, Connector_PinHeader_2.54mm:PinHeader_1x02_P2.54mm_Horizontal, F.Cu at (50.2, 31.3)
- added J5: FAN1, Connector_PinHeader_2.54mm:PinHeader_1x02_P2.54mm_Horizontal, F.Cu at (50.2, 38.5)
- added J6: FAN2, Connector_PinHeader_2.54mm:PinHeader_1x02_P2.54mm_Horizontal, F.Cu at (50.2, 45.7)
- added J7: FAN4, Connector_PinHeader_2.54mm:PinHeader_1x02_P2.54mm_Horizontal, F.Cu at (50.2, 52.9)
- added J8: T0, Connector_PinHeader_2.54mm:PinHeader_1x02_P2.54mm_Horizontal, F.Cu at (79.0, 31.3)
- added J9: T1, Connector_PinHeader_2.54mm:PinHeader_1x02_P2.54mm_Horizontal, F.Cu at (79.0, 38.5)
- added Q1: DTC143E, Package_TO_SOT_SMD:SOT-723, F.Cu at (63.1, 40.1)
- added Q2: DTC143E, Package_TO_SOT_SMD:SOT-723, F.Cu at (63.1, 43.0)
- added Q4: DTC143E, Package_TO_SOT_SMD:SOT-723, F.Cu at (63.1, 45.8)
- added Q5: DTC143E, Package_TO_SOT_SMD:SOT-723, F.Cu at (63.1, 48.6)
- added R10: 4k7, Resistor_SMD:R_0402_1005Metric, F.Cu at (66.0, 39.7)
- added R12: 10k, Resistor_SMD:R_0402_1005Metric, F.Cu at (66.0, 41.7)
- added R14: 4k7, Resistor_SMD:R_0402_1005Metric, F.Cu at (66.0, 43.6)
- added R16: 4k7, Resistor_SMD:R_0402_1005Metric, F.Cu at (66.0, 45.6)
- added R18: 4k7, Resistor_SMD:R_0402_1005Metric, F.Cu at (91.6, 30.0)
- added R19: 4k7, Resistor_SMD:R_0402_1005Metric, F.Cu at (91.6, 32.0)
- added R20: 330, Resistor_SMD:R_0402_1005Metric, F.Cu at (91.6, 34.0)
- added R21: 4k7, Resistor_SMD:R_0402_1005Metric, F.Cu at (91.6, 35.9)
- added R22: 4k7, Resistor_SMD:R_0402_1005Metric, F.Cu at (91.6, 37.9)
- added R25: 330, Resistor_SMD:R_0402_1005Metric, F.Cu at (77.2, 67.3)
- added R26: 330, Resistor_SMD:R_0402_1005Metric, F.Cu at (77.2, 69.3)
- added U4: ADS1015IDGS, Package_SO:TSSOP-10_3x3mm_P0.5mm, F.Cu at (93.6, 41.2)
- added U5: PCA9536D, Package_SO:SOIC-8_3.9x4.9mm_P1.27mm, F.Cu at (75.5, 63.1)
Other:
- board size 35 x 35 mm -> 85 x 35 mm

Commit message: tried python pcbnew, did not work
Parts:
- removed C10, C11, C7, C8, C9: 0.1µF, Capacitor_SMD:C_0402_1005Metric
- removed D2: BLUE, LED_SMD:LED_0805_2012Metric
- removed D3, D4: YELLOW, LED_SMD:LED_0805_2012Metric
- removed H5, H6, H7, H8: MountingHole_Pad, MountingHole:MountingHole_2.2mm_M2_Pad_TopBottom
- removed J10: T2, Connector_PinHeader_2.54mm:PinHeader_1x02_P2.54mm_Horizontal
- removed J11: T3, Connector_PinHeader_2.54mm:PinHeader_1x02_P2.54mm_Horizontal
- removed J12: Breakout_Board_ADXL345, Connector_PinHeader_2.54mm:PinHeader_1x04_P2.54mm_Horizontal
- removed J2: Fan_12/5V_Regelung, Connector_PinHeader_2.54mm:PinHeader_1x03_P2.54mm_Horizontal
- removed J4: FAN0, Connector_PinHeader_2.54mm:PinHeader_1x02_P2.54mm_Horizontal
- removed J5: FAN1, Connector_PinHeader_2.54mm:PinHeader_1x02_P2.54mm_Horizontal
- removed J6: FAN2, Connector_PinHeader_2.54mm:PinHeader_1x02_P2.54mm_Horizontal
- removed J7: FAN4, Connector_PinHeader_2.54mm:PinHeader_1x02_P2.54mm_Horizontal
- removed J8: T0, Connector_PinHeader_2.54mm:PinHeader_1x02_P2.54mm_Horizontal
- removed J9: T1, Connector_PinHeader_2.54mm:PinHeader_1x02_P2.54mm_Horizontal
- removed Q1, Q2, Q4, Q5: DTC143E, Package_TO_SOT_SMD:SOT-723
- removed R10, R14, R16, R18, R19, R21, R22: 4k7, Resistor_SMD:R_0402_1005Metric
- removed R12: 10k, Resistor_SMD:R_0402_1005Metric
- removed R20, R25, R26: 330, Resistor_SMD:R_0402_1005Metric
- removed U4: ADS1015IDGS, Package_SO:TSSOP-10_3x3mm_P0.5mm
- removed U5: PCA9536D, Package_SO:SOIC-8_3.9x4.9mm_P1.27mm
- moved C13 1.52 mm to (115.5, 113.0)
Routing:
- net GND: track 223.2 -> 216.2 mm
- net +5V: track 78.1 -> 83.0 mm
- net SCL: track 22.5 -> 23.6 mm
- net Net-(J1-Pin_3): track 5.85 -> 6.97 mm
- net DSCLP: track 14.4 -> 15.2 mm
- net SDA: track 19.3 -> 20.1 mm
Other:
- board size 85 x 35 mm -> 35 x 35 mm

Commit message: finished work, did not get step to convert to pdf file
Routing:
- net DSDAM: track 12.4 -> 13.3 mm
- net DSCLM: track 11.9 -> 12.8 mm
Changed lines of the file:
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@@
-	)
-	(segment
-		(start 123.02 112.420001)
-		(end 122.619999 112.02)
-		(width 0.5)
-		(layer "F.Cu")
-		(net 5)
 	)
 	(segment
@@
 	)
 	(segment
-		(start 122.619999 112.02)
-		(end 121.5 112.02)
-		(width 0.5)
-		(layer "F.Cu")
-		(net 5)
-	)
-	(segment
 		(start 119.75 130.75)
 		(end 122.05 130.75)
@@
 	)
 	(segment
+		(start 123.02 112.470001)
+		(end 122.569999 112.02)
+		(width 0.5)
+		(layer "F.Cu")
+		(net 5)
+	)
+	(segment
 		(start 121.5 112.02)
 		(end 121.5 102.3625)
@@
 	)
 	(segment
+		(start 122.569999 112.02)
+		(end 121.5 112.02)
+		(width 0.5)
+		(layer "F.Cu")
+		(net 5)
+	)
+	(segment
 		(start 121.125 126)
 		(end 119.19 126)
@@
 	)
 	(segment
+		(start 123.02 112.74)
+		(end 123.02 112.470001)
+		(width 0.5)
+		(layer "F.Cu")
+		(net 5)
+	)
+	(segment
 		(start 116 123.56)
 		(end 114.94 123.56)
@@
 		(start 121.1375 102)
 		(end 115 102)
-		(width 0.5)
-		(layer "F.Cu")
-		(net 5)
-	)
-	(segment
-		(start 123.02 112.74)
-		(end 123.02 112.420001)
 		(width 0.5)
 		(layer "F.Cu")
@@
 	)
 	(segment
-		(start 123.51 116.99)
-		(end 126 114.5)
-		(width 0.3)
-		(layer "F.Cu")
-		(net 11)
-	)
-	(segment
 		(start 129 112.75)
 		(end 126 112.75)
@@
 	)
 	(segment
-		(start 126 114.5)
-		(end 126 114.48)
+		(start 122.65 116.99)
+		(end 124.373604 116.99)
+		(width 0.3)
+		(layer "F.Cu")
+		(net 11)
+	)
+	(segment
+		(start 124.373604 116.99)
+		(end 124.75 116.613604)
+		(width 0.3)
+		(layer "F.Cu")
+		(net 11)
+	)
+	(segment
+		(start 124.75 116.613604)
+		(end 124.75 115)
 		(width 0.3)
 		(layer "F.Cu")
@@
 	)
 	(segment
+		(start 124.75 115)
+		(end 125.27 114.48)
+		(width 0.3)
+		(layer "F.Cu")
+		(net 11)
+	)
+	(segment
 		(start 126 114.48)
 		(end 128.695 114.48)
@@
 	)
 	(segment
-		(start 122.65 116.99)
-		(end 123.51 116.99)
-		(width 0.3)
-		(layer "F.Cu")
-		(net 11)
-	)
-	(segment
-		(start 124.51 117.99)
-		(end 126 119.48)
-		(width 0.3)
-		(layer "F.Cu")
-		(net 12)
+		(start 125.27 114.48)
+		(end 126 114.48)
+		(width 0.3)
+		(layer "F.Cu")
+		(net 11)
 	)
 	(segment
@@
 	)
 	(segment
+		(start 122.65 117.99)
+		(end 125.24 117.99)
+		(width 0.3)
+		(layer "F.Cu")
+		(net 12)
+	)
+	(segment
 		(start 127.5 118.75)
 		(end 129.495 118.75)
@@
 	)
 	(segment
-		(start 122.65 117.99)
-		(end 124.51 117.99)
-		(width 0.3)
-		(layer "F.Cu")
-		(net 12)
-	)
-	(segment
 		(start 121.26 112.74)
 		(end 122 112.74)
@@
 	)
 	(segment
+		(start 125.24 117.99)
+		(end 126 118.75)
+		(width 0.3)
+		(layer "F.Cu")
+		(net 12)
+	)
+	(segment
 		(start 126 119.48)
 		(end 126.77 119.48)
@@
 	)
 	(segment
+		(start 126 118.75)
+		(end 126 119.48)
+		(width 0.3)
+		(layer "F.Cu")
+		(net 12)
+	)
+	(segment
 		(start 128.555 122.24)
 		(end 129.5 121.295)
@@
 	)
 	(segment
+		(start 124.74 118.49)
+		(end 125 118.75)
+		(width 0.3)
+		(layer "F.Cu")
+		(net 13)
+	)
+	(segment
+		(start 125.25 120.5)
+		(end 126 120.5)
+		(width 0.3)
+		(layer "F.Cu")
+		(net 13)
+	)
+	(segment
+		(start 122.65 118.49)
+		(end 124.74 118.49)
+		(width 0.3)
+		(layer "F.Cu")
+		(net 13)
+	)
+	(segment
 		(start 126.75 120.5)
 		(end 127.545 121.295)
@@
 	)
 	(segment
-		(start 122.65 118.49)
-		(end 123.99 118.49)
-		(width 0.3)
-		(layer "F.Cu")
-		(net 13)
-	)
-	(segment
-		(start 123.99 118.49)
-		(end 126 120.5)
+		(start 125 118.75)
+		(end 125 120.25)
+		(width 0.3)
+		(layer "F.Cu")
+		(net 13)
+	)
+	(segment
+		(start 125 120.25)
+		(end 125.25 120.5)
 		(width 0.3)
 		(layer "F.Cu")
@@
 	)
 	(segment
-		(start 122.65 117.49)
-		(end 124.01 117.49)
-		(width 0.3)
-		(layer "F.Cu")
-		(net 14)
-	)
-	(segment
 		(start 127 115.5)
 		(end 126 115.5)
@@
 	(segment
 		(start 122.65 117.49)
+		(end 124.51 117.49)
+		(width 0.3)
+		(layer "F.Cu")
+		(net 14)
+	)
+	(segment
+		(start 126 116)
+		(end 126 115.5)
+		(width 0.3)
+		(layer "F.Cu")
+		(net 14)
+	)
+	(segment
+		(start 122.65 117.49)
 		(end 121.6825 117.49)
-		(width 0.3)
-		(layer "F.Cu")
-		(net 14)
-	)
-	(segment
-		(start 124.01 117.49)
-		(end 126 115.5)
 		(width 0.3)
 		(layer "F.Cu")
@@
 		(layer "F.Cu")
 		(net 14)
+	)
+	(segment
+		(start 124.51 117.49)
+		(end 126 116)
+		(width 0.3)
+		(layer "F.Cu")
+		(net 14)
