File: 2nd-mainboard-pcb/atmega.kicad_sch (KiCad schematic)
At the start: 31 parts, among them J10 FAN2, J11 FAN4, J2 Conn_02x03_Odd_Even, J3 T0, J4 T1, J5 T2, J6 T3, J8 FAN0, J9 FAN1, Q2 DTC143E, Q3 DTC143E, Q4 DTC143E, Q5 DTC143E, U1 ATmega328PB-A, Y1 ECS-160-18-4X-CKM

Commit message: jtag funktionalität
Parts:
- removed J2: Conn_02x03_Odd_Even, symbol Connector_Generic:Conn_02x03_Odd_Even
- removed Q2: DTC143E, Package_TO_SOT_SMD:SOT-723, symbol Transistor_BJT:DTC143E
- added D5, D6: YELLOW, LED_SMD:LED_0805_2012Metric, symbol Device:LED
- added J12: Fan_12/5V_Regelung, Connector_PinHeader_2.54mm:PinHeader_1x03_P2.54mm_Horizontal, symbol Connector:Conn_01x03_Pin
- added Q1: DTC143E, Package_TO_SOT_SMD:SOT-723, symbol Transistor_BJT:DTC143E
- added R12, R13: 330, Resistor_SMD:R_0402_1005Metric, symbol Device:R
Connections:
- net +5V: now also J12.1 (Pin_1); no longer J10.2 (Pin_2), J11.2 (Pin_2), J8.2 (Pin_2), J9.2 (Pin_2)
- net FAN_0_PWM: now also Q1.1 (B)
- net GND: now also Q1.2 (E), R12.2, R13.2
- net LED_0: now also D5.2 (A)
- net LED_1: now also D6.2 (A)
- net Quartz_1: now reaches C6.1, U1.8 (XTAL2/PB7), Y1.1
- net at J8.1 (Pin_1): now also Q1.3 (C)
- net Quartz_2: now reaches C7.1, U1.7 (XTAL1/PB6), Y1.2
- net reset renamed RESET
- new net: D6.1 (K), R13.1
- new net: D5.1 (K), R12.1
- new net +12V: J12.3 (Pin_3)
- new net Fan_Versorgung: J10.2 (Pin_2), J11.2 (Pin_2), J12.2 (Pin_2), J8.2 (Pin_2), J9.2 (Pin_2)
Other:
- moved on the sheet: C6, C7, Y1
