File: 2nd-mainboard-pcb/2nd-mainboard-pcb.kicad_pcb (KiCad board)
At the start: 2 copper layers, 50 parts, among them J1 USB_C_Receptacle, J10 FAN2, J11 FAN4, J12 Fan_12/5V_Regelung, J3 T0, J4 T1, J5 T2, J6 T3, J7 Power, J8 FAN0, J9 FAN1, Q2 DTC143E, Q3 DTC143E, Q4 DTC143E, Q5 DTC143E, SW1 SW_DIP_x01, U1 ATmega328PB-A, U2 FT232RL

Commit message: finished stacked design, annotaded
Parts:
- removed C10, C11, C12, C16, C17, C9: 0.1µF, Capacitor_SMD:C_0402_1005Metric
- removed C13, C8: 0.1µF, Capacitor_SMD:CP_Elec_5x3
- removed C14, C15: 0.22µF, Capacitor_SMD:C_0402_1005Metric
- removed D1: SMAJ5.0A, Diode_SMD:D_SMA
- removed D3: YELLOW, LED_SMD:LED_0805_2012Metric
- removed D7: GREEN, LED_SMD:LED_0805_2012Metric
- removed J1: USB_C_Receptacle, Connector_USB:USB_C_Receptacle_GCT_USB4085
- removed J12: Fan_12/5V_Regelung, Connector_PinHeader_2.54mm:PinHeader_1x03_P2.54mm_Horizontal
- removed JP1, JP2: MEASO, Jumper:SolderJumper-2_P1.3mm_Bridged_Pad1.0x1.5mm
- removed Q2, Q3, Q4, Q5: DTC143E, Package_TO_SOT_SMD:SOT-723
- removed R10, R6, R7, R9: 4k7, Resistor_SMD:R_0402_1005Metric
- removed R11, R12, R13, R8: 330, Resistor_SMD:R_0402_1005Metric
- removed SW1: SW_DIP_x01, Button_Switch_SMD:SW_SPST_EVQQ2
- removed TP2: 5V_Test, TestPoint:TestPoint_Pad_D3.0mm
- removed TP3: GND_Test, TestPoint:TestPoint_Pad_D3.0mm
- removed TP4: 3V3_Test, TestPoint:TestPoint_Pad_D3.0mm
- removed TP5: 12V_Test, TestPoint:TestPoint_Pad_D3.0mm
- added C23: 0.1µF, Capacitor_SMD:C_0402_1005Metric, F.Cu at (-77.5, -3.10)
- added C24: 0.1µF, Capacitor_SMD:C_0402_1005Metric, F.Cu at (-77.5, -1.13)
- added C25: 0.1µF, Capacitor_SMD:C_0402_1005Metric, F.Cu at (-77.5, 0.84)
- added C26: 0.1µF, Capacitor_SMD:C_0402_1005Metric, F.Cu at (-77.5, 2.81)
- added H1: MountHole, MountingHole:MountingHole_2.2mm_M2_Pad_TopBottom, F.Cu at (-100.9, 9.53)
- added H2: MountHole, MountingHole:MountingHole_2.2mm_M2_Pad_TopBottom, F.Cu at (-100.9, 15.5)
- added H3: MountHole, MountingHole:MountingHole_2.2mm_M2_Pad_TopBottom, F.Cu at (-100.9, 21.4)
- added H4: MountHole, MountingHole:MountingHole_2.2mm_M2_Pad_TopBottom, F.Cu at (-100.9, 27.4)
- added J13: Stepper Motor, Imported_Component_Footprints:JST_S4B-XH-A-1, F.Cu at (97.5, 145.0)
- added J14: Servo Motor BL Touch, Imported_Component_Footprints:JST_XH_S3B-XH-A_1x03_P2.50mm_Horizontal, F.Cu at (107.5, 141.6)
- added J2: USB_C_Receptacle, Connector_USB:USB_C_Receptacle_GCT_USB4085, F.Cu at (61.5, 127.0)
- added J20: Steckverbinder_Male_1, CustomFotLibByJan:BF100-16-A-D-1-0640-L-C, F.Cu at (-96.2, 7.63)
- added J21: Steckverbinder_Male_2, CustomFotLibByJan:BF100-16-A-D-1-0640-L-C, F.Cu at (-87.6, 7.63)
- added J22: Steckverbinder_Female_2, CustomFotLibByJan:BF030-16A-B1-0360-0277-0600-LB, F.Cu at (-78.6, 7.63)
- added R14: 330, Resistor_SMD:R_0402_1005Metric, F.Cu at (-80.4, -14.7)
- added R15: 330, Resistor_SMD:R_0402_1005Metric, F.Cu at (-80.4, -12.8)
- added R16: 4k7, Resistor_SMD:R_0402_1005Metric, F.Cu at (-80.4, -10.8)
- added R18: 4k7, Resistor_SMD:R_0402_1005Metric, F.Cu at (-80.4, -6.78)
- added R19: 4k7, Resistor_SMD:R_0402_1005Metric, F.Cu at (-80.4, -4.79)
- added R20: 1k, Resistor_SMD:R_0402_1005Metric, F.Cu at (-58.8, 2.81)
- added TP11: 3V3_Test, TestPoint:TestPoint_Pad_D3.0mm, F.Cu at (-62.7, 1.30)
- added TP12: 5V_Test, TestPoint:TestPoint_Pad_D3.0mm, F.Cu at (-62.7, 6.35)
- added TP15: GND_Test, TestPoint:TestPoint_Pad_D3.0mm, F.Cu at (-62.7, 11.4)
- added TP16: 12V_Test, TestPoint:TestPoint_Pad_D3.0mm, F.Cu at (-62.7, 16.4)
- added TP17: Netzteil_Test, TestPoint:TestPoint_Pad_D3.0mm, F.Cu at (-62.7, 21.5)
- added U10: RJK0456DPB-00-J5, Imported_Component_Footprints:RJK0456DPB_00_J5, F.Cu at (-86.1, -5.89)
- added U11: MPU-6050, Sensor_Motion:InvenSense_QFN-24_4x4mm_P0.5mm, F.Cu at (70.0, 24.5)
- added U12: TMC2209_SILENTSTEPSTICK, Imported_Component_Footprints:MODULE_TMC2209_SILENTSTEPSTICK, F.Cu at (-39.6, -27.7)
- added U3: TPS56837HRPAR, Imported_Component_Footprints:TPS56837HRPAR, F.Cu at (-50.8, 29.7)
- added U4: TPS565208, Package_TO_SOT_SMD:SOT-23-6, F.Cu at (-44.5, 26.2)
- added U5: PTS647SM38SMTR2LFS, Imported_Component_Footprints:SW_PTS647SM38SMTR2LFS_CNK, F.Cu at (-37.3, 13.1)
- added U6: FT232RL, Package_SO:SSOP-28_5.3x10.2mm_P0.65mm, F.Cu at (-48.5, 4.80)
- added U7: ATmega328PB-A, Package_QFP:TQFP-32_7x7mm_P0.8mm, F.Cu at (-73.1, -9.91)
- added U8: RJK0456DPB-00-J5, Imported_Component_Footprints:RJK0456DPB_00_J5, F.Cu at (-86.1, -12.5)
- added U9: TPM16050-S6TR, Imported_Component_Footprints:TPM16050_S6TR, F.Cu at (-87.8, -0.27)
- D6: value YELLOW -> GREEN
- J3: value T0 -> Fan_12/5V_Regelung; footprint Connector_PinHeader_2.54mm:PinHeader_1x02_P2.54mm_Horizontal -> Connector_PinHeader_2.54mm:PinHeader_1x03_P2.54mm_Horizontal
- J4: value T1 -> FAN1; footprint Connector_PinHeader_2.54mm:PinHeader_1x02_P2.54mm_Horizontal -> Imported_Component_Footprints:CONN_S2B-XH-A-1LFSN_JST
- J5: value T2 -> FAN0; footprint Connector_PinHeader_2.54mm:PinHeader_1x02_P2.54mm_Horizontal -> Imported_Component_Footprints:CONN_S2B-XH-A-1LFSN_JST
- J6: value T3 -> T0
- J7: value Power -> T1; footprint Connector_PinHeader_2.54mm:PinHeader_1x03_P2.54mm_Horizontal -> Connector_PinHeader_2.54mm:PinHeader_1x02_P2.54mm_Horizontal
- J8: value FAN0 -> T2
- J9: value FAN1 -> T3
- R17: value 1k -> 4k7
- U1: value ATmega328PB-A -> SQJ409EP-T1_GE3; footprint Package_QFP:TQFP-32_7x7mm_P0.8mm -> Imported_Component_Footprints:SQJ409EP_T1_GE3
- U2: value FT232RL -> SZ1SMB5927BT3G; footprint Package_SO:SSOP-28_5.3x10.2mm_P0.65mm -> Imported_Component_Footprints:SZ1SMB5927BT3G
- moved R17 360.3 mm to (-80.4, -8.77)
- moved J7 340.7 mm to (-101.5, -29.1)
- moved J6 336.6 mm to (-101.5, -36.3)
- moved J10 335.0 mm to (-101.5, -7.52)
- moved J11 335.0 mm to (-101.5, -0.32)
- moved J8 335.0 mm to (-101.5, -21.9)
- moved J9 335.0 mm to (-101.5, -14.7)
- moved A1 326.9 mm to (-63.2, -36.6), turned to 0 degrees
- moved D4 317.9 mm to (-73.8, -2.56)
- moved J3 316.7 mm to (-88.1, -23.1)
- moved D5 293.2 mm to (-73.8, 0.47)
- moved D6 280.8 mm to (-58.0, 0.29)
- moved U2 244.5 mm to (-43.5, 21.0)
- moved U1 238.8 mm to (-50.4, 22.3)
- moved J5 197.8 mm to (60.0, 142.5)
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Connections:
- A1 pad 1: unconnected-(A1-GND-Pad1) -> GND
- A1 pad 10: unconnected-(A1-M0-Pad10) -> M0
- A1 pad 11: unconnected-(A1-M1-Pad11) -> M1
- A1 pad 12: unconnected-(A1-M2-Pad12) -> M2
- A1 pad 13: unconnected-(A1-~{RST}-Pad13) -> +5V
- A1 pad 14: unconnected-(A1-~{SLP}-Pad14) -> +5V
- A1 pad 15: unconnected-(A1-STEP-Pad15) -> STEP
- A1 pad 16: unconnected-(A1-DIR-Pad16) -> DIR
- A1 pad 3: unconnected-(A1-A2-Pad3) -> STP_A2
- A1 pad 4: unconnected-(A1-A1-Pad4) -> STP_A1
- A1 pad 5: unconnected-(A1-B1-Pad5) -> STP_B1
- A1 pad 6: unconnected-(A1-B2-Pad6) -> STP_B2
- A1 pad 7: unconnected-(A1-GND-Pad7) -> GND
- A1 pad 8: unconnected-(A1-VMOT-Pad8) -> +12V
- D4 pad 2: IO1 -> LED_0
- D5 pad 2: LED_0 -> LED_1
- D6 pad 2: LED_1 -> +5V
- J3 pad 1: GND -> +5V_POW
- J3 pad 2: ADC0 -> Fan_Versorgung
- J4 pad 1: GND -> Net-(J4-Pin_1)
- J4 pad 2: ADC1 -> Net-(J4-Pin_2)
- J5 pad 1: GND -> Net-(J4-Pin_1)
- J5 pad 2: ADC2 -> Net-(J4-Pin_2)
- J6 pad 2: ADC3 -> ADC0
- J7 pad 1: Net-(J7-Pin_1) -> GND
- J7 pad 2: GND -> ADC1
- J8 pad 1: Net-(J8-Pin_1) -> GND
- J8 pad 2: Fan_Versorgung -> ADC2
- J9 pad 1: Net-(J9-Pin_1) -> GND
- J9 pad 2: Fan_Versorgung -> ADC3
- R17 pad 1: Net-(D7-K) -> AREF
- R17 pad 2: GND -> ADC1
- U1 pad 1: unconnected-(U1-PD3-Pad1) -> PWR_IN_PROT
- U1 pad 2: unconnected-(U1-PD4-Pad2) -> PWR_IN_PROT
- U1 pad 3: unconnected-(U1-PE0-Pad3) -> PWR_IN_PROT
- U1 pad 4: AREF -> Net-(U1-G)
- U1 pad 5: GND -> +24V
- U2 pad 1: TXD -> PWR_IN_PROT
- U2 pad 2: unconnected-(U2-DTR-Pad2) -> Net-(U1-G)

Commit message: alle bauteile hinzugefügt
Parts:
- removed D5: YELLOW, LED_SMD:LED_0805_2012Metric
- removed D6: GREEN, LED_SMD:LED_0805_2012Metric
- removed the H1 at (-100.9, 9.53)
- removed the H2 at (-100.9, 15.5)
- removed the H3 at (-100.9, 21.4)
- removed the H4 at (-100.9, 27.4)
- removed J22: Steckverbinder_Female_2, CustomFotLibByJan:BF030-16A-B1-0360-0277-0600-LB
- removed the J3 at (-88.1, -23.1)
- removed R18, R19: 4k7, Resistor_SMD:R_0402_1005Metric
- removed R20: 1k, Resistor_SMD:R_0402_1005Metric
- removed TP11: 3V3_Test, TestPoint:TestPoint_Pad_D3.0mm
- removed TP12: 5V_Test, TestPoint:TestPoint_Pad_D3.0mm
- removed TP15: GND_Test, TestPoint:TestPoint_Pad_D3.0mm
- removed TP16: 12V_Test, TestPoint:TestPoint_Pad_D3.0mm
- removed TP17: Netzteil_Test, TestPoint:TestPoint_Pad_D3.0mm
- removed the U1 at (-50.4, 22.3)
- removed U11: MPU-6050, Sensor_Motion:InvenSense_QFN-24_4x4mm_P0.5mm
- removed the U6 at (-48.5, 4.80)
- added C1: 100nF, Capacitor_SMD:C_0402_1005Metric_Pad0.74x0.62mm_HandSolder, F.Cu at (139.3, -50.1)
- added C1: 100nF, Capacitor_SMD:C_0402_1005Metric_Pad0.74x0.62mm_HandSolder, F.Cu at (165.2, 134.9)
- added C10: 100nF, Capacitor_SMD:C_0402_1005Metric_Pad0.74x0.62mm_HandSolder, F.Cu at (139.3, -44.1)
- added C11: 10µF, Capacitor_SMD:C_0805_2012Metric_Pad1.18x1.45mm_HandSolder, F.Cu at (125.2, -43.5)
- added C12: 10µF, Capacitor_SMD:C_0805_2012Metric_Pad1.18x1.45mm_HandSolder, F.Cu at (125.2, -40.5)
- added C12: 10µF, Capacitor_SMD:C_0805_2012Metric_Pad1.18x1.45mm_HandSolder, F.Cu at (171.2, 150.1)
- added C13: 100nF, Capacitor_SMD:C_0402_1005Metric_Pad0.74x0.62mm_HandSolder, F.Cu at (175.0, 138.7)
- added C13: 100nF, Capacitor_SMD:C_0402_1005Metric_Pad0.74x0.62mm_HandSolder, F.Cu at (139.3, -42.2)
- added C14: 22µF, Capacitor_SMD:C_1210_3225Metric_Pad1.33x2.70mm_HandSolder, F.Cu at (116.8, -47.3)
- added C15: 10µF, Capacitor_SMD:C_0805_2012Metric_Pad1.18x1.45mm_HandSolder, F.Cu at (195.0, -64.9)
- added C16: 100nF, Capacitor_SMD:C_0402_1005Metric_Pad0.74x0.62mm_HandSolder, F.Cu at (199.1, -65.4)
- added C17: 100nF, Capacitor_SMD:C_0402_1005Metric_Pad0.74x0.62mm_HandSolder, F.Cu at (199.1, -63.4)
- added C18: 100nF, Capacitor_SMD:C_0402_1005Metric_Pad0.74x0.62mm_HandSolder, F.Cu at (199.1, -61.5)
- added C19: 1uF, Capacitor_SMD:C_0805_2012Metric_Pad1.18x1.45mm_HandSolder, F.Cu at (195.0, -61.9)
- added C2: 22nF, Capacitor_SMD:C_1210_3225Metric_Pad1.33x2.70mm_HandSolder, F.Cu at (183.8, 156.4)
- added C2: 22nF, Capacitor_SMD:C_1210_3225Metric_Pad1.33x2.70mm_HandSolder, F.Cu at (81.5, -77.0)
- added C20: 4.7uF, Capacitor_SMD:C_0805_2012Metric_Pad1.18x1.45mm_HandSolder, F.Cu at (155.3, -73.2)
- added C21: 100nF, Capacitor_SMD:C_0402_1005Metric_Pad0.74x0.62mm_HandSolder, F.Cu at (128.8, -96.2)
- added C22: 18pF, Capacitor_SMD:C_0402_1005Metric_Pad0.74x0.62mm_HandSolder, F.Cu at (128.8, -94.2)
- added C27: 0.1µF, Capacitor_SMD:C_0402_1005Metric_Pad0.74x0.62mm_HandSolder, F.Cu at (128.8, -84.4)
- added C28: 100nF, Capacitor_SMD:C_0402_1005Metric_Pad0.74x0.62mm_HandSolder, F.Cu at (162.7, -87.5)
- added C29: 4.7uF, Capacitor_SMD:C_0805_2012Metric_Pad1.18x1.45mm_HandSolder, F.Cu at (173.0, -87.0)
- added C3: 10µF, Capacitor_SMD:C_0805_2012Metric_Pad1.18x1.45mm_HandSolder, F.Cu at (164.5, 150.2)
- added C3: 10µF, Capacitor_SMD:C_0805_2012Metric_Pad1.18x1.45mm_HandSolder, F.Cu at (125.2, -49.5)
- added C30: 100nF, Capacitor_SMD:C_0402_1005Metric_Pad0.74x0.62mm_HandSolder, F.Cu at (162.7, -85.6)
- added C31: 100nF, Capacitor_SMD:C_0402_1005Metric_Pad0.74x0.62mm_HandSolder, F.Cu at (162.7, -83.6)
- added C32: 4.7uF, Capacitor_SMD:C_0805_2012Metric_Pad1.18x1.45mm_HandSolder, F.Cu at (173.0, -84.0)
- added C33: 100nF, Capacitor_SMD:C_0402_1005Metric_Pad0.74x0.62mm_HandSolder, F.Cu at (162.7, -81.6)
- added C34: 100nF, Capacitor_SMD:C_0402_1005Metric_Pad0.74x0.62mm_HandSolder, F.Cu at (162.7, -79.7)
- added C4: 10µF, Capacitor_SMD:C_0805_2012Metric_Pad1.18x1.45mm_HandSolder, F.Cu at (125.2, -46.5)
- added C4: 10µF, Capacitor_SMD:C_0805_2012Metric_Pad1.18x1.45mm_HandSolder, F.Cu at (169.5, 150.1)
- added C5: 10µF, Capacitor_SMD:C_1210_3225Metric_Pad1.33x2.70mm_HandSolder, F.Cu at (162.8, 150.2)
- added C5: 10µF, Capacitor_SMD:C_1210_3225Metric_Pad1.33x2.70mm_HandSolder, F.Cu at (81.5, -72.8)
- added C6: 100nF, Capacitor_SMD:C_0402_1005Metric_Pad0.74x0.62mm_HandSolder, F.Cu at (139.3, -48.1)
- added C6: 100nF, Capacitor_SMD:C_0402_1005Metric_Pad0.74x0.62mm_HandSolder, F.Cu at (173.0, 150.2)
- added C7: 100nF, Capacitor_SMD:C_0402_1005Metric_Pad0.74x0.62mm_HandSolder, F.Cu at (139.3, -46.1)
- added C8: 47µF, Capacitor_SMD:C_1210_3225Metric_Pad1.33x2.70mm_HandSolder, F.Cu at (81.5, -68.5)
- added C9: 22nF, Capacitor_SMD:C_1210_3225Metric_Pad1.33x2.70mm_HandSolder, F.Cu at (81.5, -64.2)
- added D1: WE-TVSP_DO-214AA_600W_BI, Imported_Component_Footprints:824521241, F.Cu at (131.7, -40.0)
- added D1: WE-TVSP_DO-214AA_600W_BI, Imported_Component_Footprints:824521241, F.Cu at (181.6, 151.7)
- added D2: WE-TVSP_DO-214AA_600W_BI, Imported_Component_Footprints:824521241, F.Cu at (195.7, -46.4)
- added D3: YELLOW, LED_SMD:LED_0805_2012Metric, F.Cu at (150.7, -77.8)
- added H1: MountHole, MountingHole:MountingHole_2.2mm_M2_Pad_TopBottom, F.Cu at (18.5, 19.0)
- added H1: MountHole, MountingHole:MountingHole_2.2mm_M2_Pad_TopBottom, F.Cu at (162.5, 128.7)
- added H10: MountHole, MountingHole:MountingHole_2.2mm_M2_Pad_TopBottom, F.Cu at (269.5, 105.5)
- added H11: MountHole, MountingHole:MountingHole_2.2mm_M2_Pad_TopBottom, F.Cu at (240.5, 134.5)
- added H12: MountHole, MountingHole:MountingHole_2.2mm_M2_Pad_TopBottom, F.Cu at (269.5, 134.5)
- added H2: MountHole, MountingHole:MountingHole_2.2mm_M2_Pad_TopBottom, F.Cu at (47.5, 19.0)
- added H2: MountHole, MountingHole:MountingHole_2.2mm_M2_Pad_TopBottom, F.Cu at (191.5, 157.7)
- added H3: MountHole, MountingHole:MountingHole_2.2mm_M2_Pad_TopBottom, F.Cu at (18.5, 48.0)
- added H3: MountHole, MountingHole:MountingHole_2.2mm_M2_Pad_TopBottom, F.Cu at (191.5, 128.7)
- added H4: MountHole, MountingHole:MountingHole_2.2mm_M2_Pad_TopBottom, F.Cu at (47.5, 48.0)
- added H4: MountHole, MountingHole:MountingHole_2.2mm_M2_Pad_TopBottom, F.Cu at (162.5, 157.7)
- added H5: MountHole, MountingHole:MountingHole_2.2mm_M2_Pad_TopBottom, F.Cu at (243.0, 53.0)
- added H6: MountHole, MountingHole:MountingHole_2.2mm_M2_Pad_TopBottom, F.Cu at (272.0, 53.0)
- added H7: MountHole, MountingHole:MountingHole_2.2mm_M2_Pad_TopBottom, F.Cu at (243.0, 82.0)
- added H8: MountHole, MountingHole:MountingHole_2.2mm_M2_Pad_TopBottom, F.Cu at (272.0, 82.0)
- added H9: MountHole, MountingHole:MountingHole_2.2mm_M2_Pad_TopBottom, F.Cu at (240.5, 105.5)
- added J1: PJ-082BH, Imported_Component_Footprints:CUI_PJ-082BH, F.Cu at (175.0, 155.2)
- added J1: PJ-082BH, Imported_Component_Footprints:CUI_PJ-082BH, F.Cu at (71.1, 143.9)
- added J12: Stepper Motor, Imported_Component_Footprints:JST_S4B-XH-A-1, F.Cu at (260.0, 138.0)
- added J16: Steckverbinder_Male_1, CustomFotLibByJan:BF100-16-A-D-1-0640-L-C, F.Cu at (26.0, 24.5)
- added J17: Steckverbinder_Male_2, CustomFotLibByJan:BF100-16-A-D-1-0640-L-C, F.Cu at (201.0, 30.5)
- added J18: Steckverbinder_Female_2, CustomFotLibByJan:BF030-16A-B1-0360-0277-0600-LB, F.Cu at (249.5, 56.8)
- added J19: Steckverbinder_Male_2, CustomFotLibByJan:BF100-16-A-D-1-0640-L-C, F.Cu at (136.3, 85.7)
- added J3: FAN0, Imported_Component_Footprints:CONN_S2B-XH-A-1LFSN_JST, F.Cu at (189.0, 139.4)
- added J3: FAN0, Imported_Component_Footprints:CONN_S2B-XH-A-1LFSN_JST, F.Cu at (24.2, 47.2)
- added JP1: MEASO, Jumper:SolderJumper-2_P1.3mm_Bridged_Pad1.0x1.5mm, F.Cu at (173.5, 141.7)
- added JP2: MEASO, Jumper:SolderJumper-2_P1.3mm_Bridged_Pad1.0x1.5mm, F.Cu at (175.5, 149.9)
- added JP3: MEASO, Jumper:SolderJumper-2_P1.3mm_Bridged_Pad1.0x1.5mm, F.Cu at (167.0, 149.9)
- added L1: 4.7µH, Imported_Component_Footprints:SPM10040T_4R7M_HZ, F.Cu at (101.0, -72.0)
- added L2: 3.3µH, Imported_Component_Footprints:IHLP2525CZER3R3M11, F.Cu at (133.1, -46.8)
- added P1: USB_C_Plug_USB2.0, Connector_USB:USB_C_Receptacle_GCT_USB4085, F.Cu at (79.7, 139.7)
- added R1: 100k, Resistor_SMD:R_0402_1005Metric, F.Cu at (185.2, 151.7)
- added R1: 100k, Resistor_SMD:R_0402_1005Metric, F.Cu at (86.0, -78.1)
- added R10: 5k1, Resistor_SMD:R_0402_1005Metric, F.Cu at (201.3, -46.0)
- added R11: 10k, Resistor_SMD:R_0402_1005Metric, F.Cu at (201.3, -44.0)
- added R12: 4k7, Resistor_SMD:R_0402_1005Metric, F.Cu at (140.5, -90.0)
- added R13: 4k7, Resistor_SMD:R_0402_1005Metric, F.Cu at (140.5, -88.0)
- added R2: 100k, Resistor_SMD:R_0402_1005Metric, F.Cu at (86.0, -76.1)
- added R2: 100k, Resistor_SMD:R_0402_1005Metric, F.Cu at (178.0, 140.2)
- added R3: 30k, Resistor_SMD:R_0402_1005Metric, F.Cu at (86.0, -74.2)
- added R3: 30k, Resistor_SMD:R_0402_1005Metric, F.Cu at (178.0, 146.2)
- added R4: 1k58, Resistor_SMD:R_0402_1005Metric, F.Cu at (86.0, -72.2)
- added R4: 1k58, Resistor_SMD:R_0402_1005Metric, F.Cu at (182.0, 146.2)
- added R5: 30.1k, Resistor_SMD:R_0402_1005Metric, F.Cu at (185.5, 145.7)
- added R5: 30.1k, Resistor_SMD:R_0402_1005Metric, F.Cu at (86.0, -70.2)
- added R6: 10, Resistor_SMD:R_0402_1005Metric, F.Cu at (185.5, 148.4)
- added R6: 10, Resistor_SMD:R_0402_1005Metric, F.Cu at (86.0, -68.2)
- added R7: 54.9k, Resistor_SMD:R_0402_1005Metric, F.Cu at (182.0, 140.2)
- added R7: 54.9k, Resistor_SMD:R_0402_1005Metric, F.Cu at (86.0, -66.2)
- added R8: 10k, Resistor_SMD:R_0402_1005Metric, F.Cu at (185.5, 140.7)
- added R8: 10k, Resistor_SMD:R_0402_1005Metric, F.Cu at (121.3, -51.5)
- added R9: 5k1, Resistor_SMD:R_0402_1005Metric, F.Cu at (201.3, -48.0)
- added R9: 5k1, Resistor_SMD:R_0402_1005Metric, F.Cu at (185.5, 137.9)
- added U1: SQJ409EP-T1_GE3, Imported_Component_Footprints:SQJ409EP_T1_GE3, F.Cu at (180.0, 143.2)
- added U1: SQJ409EP-T1_GE3, Imported_Component_Footprints:SQJ409EP_T1_GE3, F.Cu at (144.2, -46.9)
- added U6: PTS647SM38SMTR2LFS, Imported_Component_Footprints:SW_PTS647SM38SMTR2LFS_CNK, F.Cu at (166.2, 143.2)
- added U6: PTS647SM38SMTR2LFS, Imported_Component_Footprints:SW_PTS647SM38SMTR2LFS_CNK, F.Cu at (197.5, -52.1)
- added Y1: ECS-160-18-4X-CKM, Imported_Component_Footprints:XTAL_ECS-160-18-4X-CKM, F.Cu at (91.9, -99.5)
- C23: value 0.1µF -> 18pF; footprint Capacitor_SMD:C_0402_1005Metric -> Capacitor_SMD:C_0402_1005Metric_Pad0.74x0.62mm_HandSolder
- C24, C25, C26: footprint Capacitor_SMD:C_0402_1005Metric -> Capacitor_SMD:C_0402_1005Metric_Pad0.74x0.62mm_HandSolder
- J10: value FAN2 -> T3; footprint Connector_PinHeader_2.54mm:PinHeader_1x02_P2.54mm_Horizontal -> Imported_Component_Footprints:665102131822
- J11: value FAN4 -> Servo Motor SM; footprint Connector_PinHeader_2.54mm:PinHeader_1x02_P2.54mm_Horizontal -> Imported_Component_Footprints:JST_XH_S3B-XH-A_1x03_P2.50mm_Horizontal
- J13: value Stepper Motor -> Steckverbinder_Male_1; footprint Imported_Component_Footprints:JST_S4B-XH-A-1 -> CustomFotLibByJan:BF100-16-A-D-1-0640-L-C
- J14: value Servo Motor BL Touch -> Microstepping; footprint Imported_Component_Footprints:JST_XH_S3B-XH-A_1x03_P2.50mm_Horizontal -> Imported_Component_Footprints:FTSH-103-01-L-DH
- J2: value USB_C_Receptacle -> Fan_12/5V_Regelung; footprint Connector_USB:USB_C_Receptacle_GCT_USB4085 -> Imported_Component_Footprints:FTS_103_01_F_S
- J20: value Steckverbinder_Male_1 -> Steckverbinder_Female_2; footprint CustomFotLibByJan:BF100-16-A-D-1-0640-L-C -> CustomFotLibByJan:BF030-16A-B1-0360-0277-0600-LB
- J21: value Steckverbinder_Male_2 -> ISP; footprint CustomFotLibByJan:BF100-16-A-D-1-0640-L-C -> Imported_Component_Footprints:FTSH-103-01-L-DH
- J5: value FAN0 -> FAN2
- J6: value T0 -> FAN3; footprint Connector_PinHeader_2.54mm:PinHeader_1x02_P2.54mm_Horizontal -> Imported_Component_Footprints:CONN_S2B-XH-A-1LFSN_JST
- J7: value T1 -> T2; footprint Connector_PinHeader_2.54mm:PinHeader_1x02_P2.54mm_Horizontal -> Imported_Component_Footprints:665102131822
- J8: footprint Connector_PinHeader_2.54mm:PinHeader_1x02_P2.54mm_Horizontal -> Imported_Component_Footprints:665102131822
- J9: value T3 -> T2; footprint Connector_PinHeader_2.54mm:PinHeader_1x02_P2.54mm_Horizontal -> Imported_Component_Footprints:665102131822
- R14, R15: value 330 -> 4k7
- R16, R17: value 4k7 -> 330
- U10: value RJK0456DPB-00-J5 -> ATmega328PB-A; footprint Imported_Component_Footprints:RJK0456DPB_00_J5 -> Package_QFP:TQFP-32_7x7mm_P0.8mm
- U12: value TMC2209_SILENTSTEPSTICK -> MPU-6050; footprint Imported_Component_Footprints:MODULE_TMC2209_SILENTSTEPSTICK -> Sensor_Motion:InvenSense_QFN-24_4x4mm_P0.5mm
- U5: value PTS647SM38SMTR2LFS -> FT232RL; footprint Imported_Component_Footprints:SW_PTS647SM38SMTR2LFS_CNK -> Package_SO:SSOP-28_5.3x10.2mm_P0.65mm
- U7: value ATmega328PB-A -> TPM16050-S6TR; footprint Package_QFP:TQFP-32_7x7mm_P0.8mm -> Imported_Component_Footprints:TPM16050_S6TR
- U9: value TPM16050-S6TR -> RJK0456DPB-00-J5; footprint Imported_Component_Footprints:TPM16050_S6TR -> Imported_Component_Footprints:RJK0456DPB_00_J5
- moved J21 423.1 mm to (321.2, 116.5)
- moved J11 390.1 mm to (268.6, 123.0), turned to 90 degrees
- moved A1 345.9 mm to (241.6, 126.8), turned to 90 degrees
- moved J9 332.3 mm to (203.9, 116.2)
- moved U10 247.0 mm to (147.8, -85.2)
- moved J14 244.6 mm to (192.5, -87.8)
- moved J8 243.1 mm to (127.0, 61.0), turned to 180 degrees
- moved U9 239.0 mm to (134.7, -87.4)
- moved U7 238.3 mm to (155.6, -77.0)
- moved J20 237.6 mm to (121.4, 103.0)
- moved D4 235.9 mm to (150.7, -74.8)
- moved U8 235.4 mm to (134.7, -93.9)
- moved U5 232.1 mm to (186.3, -49.1)
- moved R14 232.1 mm to (140.5, -86.0)
- moved R15 232.1 mm to (140.5, -84.0)
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Connections:
- A1 pad 13: +5V -> +5V_POW
- A1 pad 14: +5V -> +5V_POW
- C23 pad 1: ADC0 -> Quartz_2
- C24 pad 1: ADC1 -> ADC0
- C25 pad 1: ADC2 -> ADC1
- C26 pad 1: ADC3 -> ADC2
- D4 pad 2: LED_0 -> LED_1
- J10 pad 1: Net-(J10-Pin_1) -> GND
- J10 pad 2: Fan_Versorgung -> ADC3
- J11 pad 1: Net-(J11-Pin_1) -> GND
- J11 pad 2: Fan_Versorgung -> +5V_POW
- J20 pad a1: SM_Servo -> MOSI
- J4 pad 1: Net-(J4-Pin_1) -> Net-(U7-OUT1)
- J4 pad 2: Net-(J4-Pin_2) -> Net-(U7-OUT2)
- J5 pad 1: Net-(J4-Pin_1) -> Fan_Versorgung
- J5 pad 2: Net-(J4-Pin_2) -> Net-(U8-D)
- J6 pad 1: GND -> Fan_Versorgung
- J6 pad 2: ADC0 -> Net-(U9-D)
- J7 pad 2: ADC1 -> ADC0
- J8 pad 2: ADC2 -> ADC1
- J9 pad 2: ADC3 -> ADC2
- R14 pad 1: Net-(D4-K) -> AREF
- R14 pad 2: GND -> ADC2
- R15 pad 1: Net-(D5-K) -> AREF
- R15 pad 2: GND -> ADC3
- R16 pad 1: AREF -> Net-(D3-K)
- R16 pad 2: ADC0 -> GND
- R17 pad 1: AREF -> Net-(D4-K)
- R17 pad 2: ADC1 -> GND
- U10 pad 1: GND -> BLT_Servo
- U10 pad 2: GND -> BLT_Switch
- U10 pad 3: GND -> LED_0
- U10 pad 4: FAN_3_PWM -> +5V_POW
- U10 pad 5: Net-(J11-Pin_1) -> GND
- U12 pad 1: GND -> unconnected-(U12-CLKIN-Pad1)
- U12 pad 10: STEP -> unconnected-(U12-REGOUT-Pad10)
- U12 pad 13: unconnected-(U12-SPRD-Pad13) -> +5V_POW
- U12 pad 14: M2 -> unconnected-(U12-NC-Pad14)
- U12 pad 15: M1 -> unconnected-(U12-NC-Pad15)
- U12 pad 18: unconnected-(U12-DIAG-Pad18) -> GND
- U12 pad 2: +5V_POW -> unconnected-(U12-NC-Pad2)
- U12 pad 3: STP_B1 -> unconnected-(U12-NC-Pad3)
- U12 pad 4: STP_A1 -> unconnected-(U12-NC-Pad4)
- U12 pad 5: STP_A2 -> unconnected-(U12-NC-Pad5)
- U12 pad 6: STP_B2 -> unconnected-(U12-AUX_DA-Pad6)
- U12 pad 7: GND -> unconnected-(U12-AUX_CL-Pad7)
- U12 pad 8: +12V -> +5V_POW
- U12 pad 9: DIR -> unconnected-(U12-AD0-Pad9)
- U5 pad 1: GND -> TXD
- U5 pad 4: RESET -> +5V_POW
- U7 pad 1: BLT_Servo -> Net-(U7-OUT2)
- U7 pad 2: BLT_Switch -> GND
- U7 pad 3: unconnected-(U7-PE0-Pad3) -> Net-(U7-OUT1)
- U7 pad 4: +5V_POW -> Fan_Versorgung
- U7 pad 5: GND -> FAN_01_PWM_counterclockwise
- U7 pad 6: unconnected-(U7-PE1-Pad6) -> FAN_01_PWM_clockwise
- U8 pad 5: Net-(J10-Pin_1) -> Net-(U8-D)
- U9 pad 1: Net-(J4-Pin_1) -> GND
- U9 pad 3: Net-(J4-Pin_2) -> GND
- U9 pad 4: Fan_Versorgung -> FAN_3_PWM
- U9 pad 5: FAN_01_PWM_counterclockwise -> Net-(U9-D)
Routing:
- net (no net): track 0.00 -> 142.3 mm
- net GND: track 0.00 -> 36.6 mm
- net +12V: track 0.00 -> 31.6 mm
- net SCL: track 0.00 -> 19.5 mm
- net SDA: track 0.00 -> 19.4 mm
- net Net-(U4-VFB): track 0.00 -> 12.5 mm
- net AREF: track 0.00 -> 12.4 mm
- net unconnected-(U6-Pad3): track 0.00 -> 4.70 mm
- net Net-(U1-G): track 0.00 -> 2.96 mm
- added copper zone on B.Cu, net GND
- added copper zone on F.Cu, net GND
Other:
- board outline added: 35 x 35 mm

Commit message: module 1 positioniert
Parts:
- removed A1: Pololu_Breakout_DRV8825, Module:Pololu_Breakout-16_15.2x20.3mm
- removed the C1 at (165.2, 134.9)
- removed the C12 at (125.2, -40.5)
- removed the C12 at (171.2, 150.1)
- removed the C13 at (175.0, 138.7)
- removed the C13 at (139.3, -42.2)
- removed the C2 at (183.8, 156.4)
- removed C24, C25, C26, C27: 0.1µF, Capacitor_SMD:C_0402_1005Metric_Pad0.74x0.62mm_HandSolder
- removed C28, C30, C31, C33, C34: 100nF, Capacitor_SMD:C_0402_1005Metric_Pad0.74x0.62mm_HandSolder
- removed C29, C32: 4.7uF, Capacitor_SMD:C_0805_2012Metric_Pad1.18x1.45mm_HandSolder
- removed the C3 at (164.5, 150.2)
- removed the C4 at (169.5, 150.1)
- removed the C5 at (162.8, 150.2)
- removed the C6 at (173.0, 150.2)
- removed the D1 at (181.6, 151.7)
- removed H1 (x2), H10, H11, H12, H2 (x2), H3 (x2), H4 (x2), H9: MountHole, MountingHole:MountingHole_2.2mm_M2_Pad_TopBottom
- removed the J1 at (175.0, 155.2)
- removed J10: T3, Imported_Component_Footprints:665102131822
- removed J11: Servo Motor SM, Imported_Component_Footprints:JST_XH_S3B-XH-A_1x03_P2.50mm_Horizontal
- removed J12: Stepper Motor, Imported_Component_Footprints:JST_S4B-XH-A-1
- removed J13, J16: Steckverbinder_Male_1, CustomFotLibByJan:BF100-16-A-D-1-0640-L-C
- removed J14: Microstepping, Imported_Component_Footprints:FTSH-103-01-L-DH
- removed J19: Steckverbinder_Male_2, CustomFotLibByJan:BF100-16-A-D-1-0640-L-C
- removed J2: Fan_12/5V_Regelung, Imported_Component_Footprints:FTS_103_01_F_S
- removed J20: Steckverbinder_Female_2, CustomFotLibByJan:BF030-16A-B1-0360-0277-0600-LB
- removed J21: ISP, Imported_Component_Footprints:FTSH-103-01-L-DH
- removed J3 (x2): FAN0, Imported_Component_Footprints:CONN_S2B-XH-A-1LFSN_JST
- removed J4: FAN1, Imported_Component_Footprints:CONN_S2B-XH-A-1LFSN_JST
- removed J5: FAN2, Imported_Component_Footprints:CONN_S2B-XH-A-1LFSN_JST
- removed J6: FAN3, Imported_Component_Footprints:CONN_S2B-XH-A-1LFSN_JST
- removed J7, J8, J9: T2, Imported_Component_Footprints:665102131822
- removed JP1, JP2, JP3: MEASO, Jumper:SolderJumper-2_P1.3mm_Bridged_Pad1.0x1.5mm
- removed the R1 at (185.2, 151.7)
- removed R12, R13, R14, R15: 4k7, Resistor_SMD:R_0402_1005Metric
- removed the R2 at (178.0, 140.2)
- removed the R3 at (178.0, 146.2)
- removed the R4 at (182.0, 146.2)
- removed the R5 at (185.5, 145.7)
- removed the R6 at (185.5, 148.4)
- removed the R7 at (182.0, 140.2)
- removed the R7 at (86.0, -66.2)
- removed the R8 at (185.5, 140.7)
- removed the R8 at (121.3, -51.5)
- removed the R9 at (185.5, 137.9)
- removed the U1 at (180.0, 143.2)
- removed U12: MPU-6050, Sensor_Motion:InvenSense_QFN-24_4x4mm_P0.5mm
- removed the U6 at (166.2, 143.2)
- removed U7: TPM16050-S6TR, Imported_Component_Footprints:TPM16050_S6TR
- removed U8, U9: RJK0456DPB-00-J5, Imported_Component_Footprints:RJK0456DPB_00_J5
- added C12: 10µF, Capacitor_SMD:C_0805_2012Metric_Pad1.18x1.45mm_HandSolder, F.Cu at (44.4, 47.2)
- added C13: 100nF, Capacitor_SMD:C_0402_1005Metric_Pad0.74x0.62mm_HandSolder, F.Cu at (44.5, 49.0)
- added R7: 54.9k, Resistor_SMD:R_0402_1005Metric, F.Cu at (43.6, 35.7)
- added R8: 10k, Resistor_SMD:R_0402_1005Metric, F.Cu at (43.6, 36.9)
- C1, C15, C16, C17, C18, C19, C2, C21, C3, C4, C5, C6, C7, C8, C9, D2, L1, R1, R11, R2, R3, R4, R5, R6, U10, U3, Y1: moved to B.Cu
- J17: value Steckverbinder_Male_2 -> Steckverbinder_Male_Leistung; moved to B.Cu
- J18: value Steckverbinder_Female_2 -> Steckverbinder_Female_Leistung
- moved H5 212.6 mm to (31.7, 29.7)
- moved H6 212.6 mm to (60.7, 29.7)
- moved H7 212.6 mm to (31.7, 58.7)
- moved H8 212.6 mm to (60.7, 58.7)
- moved J18 211.6 mm to (39.2, 33.1)
- moved C16 205.9 mm to (32.1, 55.1)
- moved C17 201.6 mm to (31.4, 48.4), turned to 180 degrees
- moved R9 199.6 mm to (30.6, 55.3), turned to 180 degrees
- moved C18 199.5 mm to (31.4, 46.7), turned to 180 degrees
- moved C19 198.7 mm to (32.0, 51.7), turned to 90 degrees
- moved C15 197.4 mm to (35.8, 51.7), turned to 90 degrees
- moved R10 196.1 mm to (33.5, 55.3), turned to 180 degrees
- moved D2 181.9 mm to (42.3, 51.2)
- moved U5 179.6 mm to (35.7, 48.7), turned to -90 degrees
- moved U6 171.7 mm to (60.7, 51.6), turned to 90 degrees
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Routing:
- net (no net): track 142.3 -> 0.00 mm
- net GND: track 36.6 -> 0.00 mm
- net +12V: track 31.6 -> 0.00 mm
- net SCL: track 19.5 -> 0.00 mm
- net SDA: track 19.4 -> 0.00 mm
- net Net-(U4-VFB): track 12.5 -> 0.00 mm
- net AREF: track 12.4 -> 0.00 mm
- net unconnected-(U6-Pad3): track 4.70 -> 0.00 mm
- net Net-(U1-G): track 2.96 -> 0.00 mm
Other:
- board outline removed

Commit message: mehr positioning
Parts:
- moved J17 14.9 mm to (39.2, 28.4), turned to -90 degrees
- moved R2 1.20 mm to (59.1, 47.6)
- moved R4 0.50 mm to (60.3, 47.6)
- moved U2 0.39 mm to (60.9, 43.8)
- moved R5 0.10 mm to (61.5, 47.6)
Routing:
- net Net-(U3-SS): track 0.00 -> 13.2 mm, vias 0 -> 2
- net Net-(U3-SW): track 0.00 -> 12.3 mm
- net PWR_IN_PROT: track 0.00 -> 2.47 mm, vias 0 -> 1
- net Net-(U3-BOOT): track 0.00 -> 2.08 mm
- net RESET: vias 0 -> 1
- removed copper zone on B.Cu, net GND
- removed copper zone on F.Cu, net GND
