File: 2nd-mainboard-pcb/2nd-mainboard-pcb - Copy.kicad_pcb (KiCad board)
At the start: 2 copper layers, 84 parts, among them J1 PJ-082BH, J12 Steckverbinder_Male_Fans, J13 Steckverbinder_Female_Leistung, J14 Steckverbinder_Male_Leistung, J16 ISP, J19 T2, J2 Fan_12/5V_Regelung, J20 T2, J21 T2, J22 T3, J3 FAN0, J4 FAN1, J5 FAN2, J6 FAN3, P1 USB_C_Plug_USB2.0, U1 SQJ409EP-T1_GE3, U10 ATmega328PB-A, U2 SZ1SMB5927BT3G, U3 TPS56837HRPAR, U4 TPS565208, U5 FT232RL, U6 PTS647SM38SMTR2LFS, U7 TPM16050-S6TR, U8 RJK0456DPB-00-J5, U9 RJK0456DPB-00-J5, Y1 ECS-160-18-4X-CKM

Commit message: Fan-PCB-Beginning
Parts:
- removed C30, C31, C32, C33, C35: 0.1µF, Capacitor_SMD:C_0402_1005Metric_Pad0.74x0.62mm_HandSolder
- removed D6: YELLOW, LED_SMD:LED_0805_2012Metric
- removed H1, H2, H3, H4: MountHole, MountingHole:MountingHole_2.2mm_M2_Pad_TopBottom
- removed J12: Steckverbinder_Male_Fans, Imported_Component_Footprints:SAMTEC_TSM-107-04-L-DV
- removed J19, J20, J21: T2, Imported_Component_Footprints:665102131822
- removed J2: Fan_12/5V_Regelung, Imported_Component_Footprints:FTS_103_01_F_S
- removed J22: T3, Imported_Component_Footprints:665102131822
- removed J3: FAN0, Imported_Component_Footprints:CONN_S2B-XH-A-1LFSN_JST
- removed J4: FAN1, Imported_Component_Footprints:CONN_S2B-XH-A-1LFSN_JST
- removed J5: FAN2, Imported_Component_Footprints:CONN_S2B-XH-A-1LFSN_JST
- removed J6: FAN3, Imported_Component_Footprints:CONN_S2B-XH-A-1LFSN_JST
- removed R15: 330, Resistor_SMD:R_0402_1005Metric
- removed R22, R23, R24, R25, R27: 4k7, Resistor_SMD:R_0402_1005Metric
- removed TH2: Thermistor_NTC, Resistor_SMD:R_0805_2012Metric
- removed U7: TPM16050-S6TR, Imported_Component_Footprints:TPM16050_S6TR
- removed U8, U9: RJK0456DPB-00-J5, Imported_Component_Footprints:RJK0456DPB_00_J5
Other:
- board text removed: "Steckverbinder_Male_2"
