File: 2nd-mainboard-pcb/usbc.kicad_sch (KiCad schematic)
At the start: 11 parts, among them P1 USB_C_Receptacle_USB2.0_14P, U5 FT232RL, U6 PTS647SM38SMTR2LFS

Commit message: stacked pcb reworked
Other:
- moved on the sheet: D2
Changed lines of the file:
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@@
+	)
+	(junction
+		(at 76.2 29.21)
+		(diameter 0)
+		(color 0 0 0 0)
 	)
 	(junction
@@
 	)
 	(junction
+		(at 96.52 148.59)
+		(diameter 0)
+		(color 0 0 0 0)
+	)
+	(junction
 		(at 63.5 29.21)
 		(diameter 0)
@@
 		(color 0 0 0 0)
 	)
-	(junction
-		(at 71.12 29.21)
-		(diameter 0)
-		(color 0 0 0 0)
-	)
 	(no_connect
 		(at 210.82 72.39)
@@
 	(wire
 		(pts
+			(xy 76.2 29.21) (xy 115.57 29.21)
+		)
+		(stroke
+			(width 0)
+			(type default)
+		)
+	)
+	(wire
+		(pts
 			(xy 82.55 148.59) (xy 96.52 148.59)
 		)
@@
 	(wire
 		(pts
-			(xy 63.5 29.21) (xy 71.12 29.21)
+			(xy 63.5 29.21) (xy 76.2 29.21)
+		)
+		(stroke
+			(width 0)
+			(type default)
+		)
+	)
+	(wire
+		(pts
+			(xy 96.52 148.59) (xy 101.6 148.59)
 		)
 		(stroke
@@
 	(wire
 		(pts
+			(xy 96.52 142.24) (xy 96.52 148.59)
+		)
+		(stroke
+			(width 0)
+			(type default)
+		)
+	)
+	(wire
+		(pts
 			(xy 166.37 64.77) (xy 170.18 64.77)
 		)
@@
 	(wire
 		(pts
-			(xy 115.57 29.21) (xy 71.12 29.21)
-		)
-		(stroke
-			(width 0)
-			(type default)
-		)
-	)
-	(wire
-		(pts
 			(xy 68.58 53.34) (xy 68.58 55.88)
 		)
@@
 	(wire
 		(pts
-			(xy 71.12 43.18) (xy 71.12 45.72)
+			(xy 76.2 43.18) (xy 76.2 45.72)
 		)
 		(stroke
@@
 	(wire
 		(pts
-			(xy 71.12 30.48) (xy 71.12 29.21)
+			(xy 76.2 30.48) (xy 76.2 29.21)
 		)
 		(stroke
@@
 	(wire
 		(pts
-			(xy 96.52 148.59) (xy 96.52 142.24)
-		)
-		(stroke
-			(width 0)
-			(type default)
-		)
-	)
-	(wire
-		(pts
 			(xy 217.17 54.61) (xy 210.82 54.61)
 		)
@@
 	(wire
 		(pts
-			(xy 71.12 45.72) (xy 101.6 45.72)
+			(xy 76.2 45.72) (xy 101.6 45.72)
 		)
 		(stroke
@@
 	(global_label "RESET"
 		(shape input)
-		(at 96.52 148.59 0)
+		(at 101.6 148.59 0)
 		(fields_autoplaced yes)
 		(effects
@@
 		)
 		(property "Intersheetrefs" "${INTERSHEET_REFS}"
-			(at 105.2503 148.59 0)
+			(at 110.3303 148.59 0)
 			(effects
 				(font
@@
 	(symbol
 		(lib_id "Imported_Component_Symbols:WE-TVSP_DO-214AA_600W_BI")
-		(at 71.12 38.1 90)
+		(at 76.2 38.1 90)
 		(unit 1)
 		(exclude_from_sim no)
@@
 		(dnp no)
 		(property "Reference" "D2"
-			(at 74.93 35.5599 90)
+			(at 80.01 35.5599 90)
 			(effects
 				(font
@@
 		)
 		(property "Value" "WE-TVSP_DO-214AA_600W_BI"
-			(at 74.93 38.0999 90)
+			(at 80.01 38.0999 90)
 			(effects
 				(font
@@
 		)
 		(property "Footprint" "Imported_Component_Footprints:824521241"
-			(at 66.548 38.1 0)
+			(at 71.628 38.1 0)
 			(effects
 				(font
@@
 		)
 		(property "Datasheet" ""
-			(at 71.12 38.1 0)
+			(at 76.2 38.1 0)
 			(effects
 				(font
@@
 		)
 		(property "Description" ""
-			(at 71.12 38.1 0)
-			(effects
-				(font
+			(at 76.2 38.1 0)
+			(effects
+				(font
