File: 2nd-mainboard-pcb/_autosave-2nd-mainboard-pcb.kicad_pcb (KiCad board)
At the start: 4 copper layers, 99 x 97.5 mm, 132 parts, among them J1 PJ-082BH, J10 Servo Motor BL Touch, J11 T3, J12 Steckverbinder_Male_Fans, J13 Steckverbinder_Female_Leistung, J14 FAN3, J15 Steckverbinder_Female_Motoren, J16 ISP, J18 Quartz, J19 T2, J2 Fan_12/5V_Regelung, J20 T2, J21 T2, J22 T3, J23 Conn_01x04_Socket, J24 Steckverbinder_Male_Leistung, J3 Fan_12/5V_Regelung, J4 FAN0, J5 FAN1, J6 FAN2, J7 Stepper Motor, J8 Servo Motor SM, J9 Microstepping, P1 USB_C_Receptacle_USB2.0_14P, U1 SQJ409EP-T1_GE3, U10 ATmega328PB-A, U12 MPU-6050, U2 SZ1SMB5927BT3G, U3 TPS56837HRPAR, U4 TPS565208, U5 FT232RL, U6 PTS647SM38SMTR2LFS, U7 TPM16050-S6TR, U8 RJK0456DPB-00-J5, U9 RJK0456DPB-00-J5, Y1 ECS-160-18-4X-CKM

Commit message: rearragned componentens
Parts:
- removed C3: 10µF, Capacitor_SMD:C_0805_2012Metric_Pad1.18x1.45mm_HandSolder
- C1, C16, C17: footprint Capacitor_SMD:C_0402_1005Metric_Pad0.74x0.62mm_HandSolder -> Capacitor_SMD:C_0603_1608Metric_Pad1.08x0.95mm_HandSolder
- C2: value 22nF -> 150pF
- moved R6 4.90 mm to (121.0, 143.7), turned to 180 degrees
- moved C7 3.95 mm to (123.9, 142.1), turned to 0 degrees
- moved C2 3.90 mm to (131.1, 118.3)
- moved C9 3.01 mm to (134.5, 118.3)
- moved R9 2.45 mm to (113.2, 143.0), turned to -90 degrees
- moved C5 1.40 mm to (134.4, 133.8)
- moved C16 1.14 mm to (114.8, 143.0), turned to -90 degrees
- moved R1 1.12 mm to (123.0, 138.3), turned to 90 degrees
- moved C4 0.80 mm to (133.8, 137.2)
- moved C17 0.80 mm to (116.5, 143.0), turned to -90 degrees
- moved C6 0.65 mm to (136.4, 138.7)
- moved R3 0.60 mm to (133.3, 121.8)
- moved R5 0.57 mm to (135.7, 130.1)
- moved C1 0.42 mm to (134.3, 123.8)
- moved R2 0.30 mm to (132.5, 130.2)
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