File: 2nd-mainboard-pcb/_autosave-2nd-mainboard-pcb_old.kicad_pcb (KiCad board)
At the start: 4 copper layers, 99 x 97.5 mm, 132 parts, among them J1 PJ-082BH, J10 Servo Motor BL Touch, J11 T3, J12 Steckverbinder_Male_Fans, J13 Steckverbinder_Female_Leistung, J14 FAN3, J15 Steckverbinder_Female_Motoren, J16 ISP, J18 Quartz, J19 T2, J2 Fan_12/5V_Regelung, J20 T2, J21 T2, J22 T3, J23 Conn_01x04_Socket, J24 Steckverbinder_Male_Leistung, J3 Fan_12/5V_Regelung, J4 FAN0, J5 FAN1, J6 FAN2, J7 Stepper Motor, J8 Servo Motor SM, J9 Microstepping, P1 USB_C_Receptacle_USB2.0_14P, U1 SQJ409EP-T1_GE3, U10 ATmega328PB-A, U12 MPU-6050, U2 SZ1SMB5927BT3G, U3 TPS56837HRPAR, U4 TPS565208, U5 FT232RL, U6 PTS647SM38SMTR2LFS, U7 TPM16050-S6TR, U8 RJK0456DPB-00-J5, U9 RJK0456DPB-00-J5, Y1 ECS-160-18-4X-CKM

Commit message: rearragned componentens
Parts:
- C13, C20, C21, C22, C23, C26, C27, C29, C30, C31, C32, C33, C35, C37, C38, C6, C7: footprint Capacitor_SMD:C_0603_1608Metric_Pad1.08x0.95mm_HandSolder -> Capacitor_SMD:C_0402_1005Metric_Pad0.74x0.62mm_HandSolder
- C28: footprint Capacitor_SMD:C_0603_1608Metric_Pad1.08x0.95mm_HandSolder -> Capacitor_SMD:C_0805_2012Metric_Pad1.18x1.45mm_HandSolder
- C8: moved to B.Cu
- R1, R10, R11, R12, R13, R14, R15, R16, R17, R22, R23, R24, R25, R4, R5, R6, R7, R8, R9: footprint Resistor_SMD:R_0603_1608Metric_Pad0.98x0.95mm_HandSolder -> Resistor_SMD:R_0402_1005Metric
- R2: footprint Resistor_SMD:R_0603_1608Metric_Pad0.98x0.95mm_HandSolder -> Resistor_SMD:R_0603_1608Metric
- R3: footprint Resistor_SMD:R_0603_1608Metric_Pad0.98x0.95mm_HandSolder -> Resistor_SMD:R_0402_1005Metric; moved to F.Cu
- moved G*** 86.9 mm to (139.7, 61.6)
- moved G*** 86.9 mm to (107.4, 82.0)
- moved R3 7.12 mm to (130.8, 114.9), turned to 180 degrees
- moved C8 5.71 mm to (131.0, 113.2), turned to 90 degrees
- moved C9 4.25 mm to (135.8, 118.5)
- moved J16 3.43 mm to (142.4, 143.3), turned to 90 degrees
- moved C2 2.75 mm to (132.2, 118.5)
- moved C30 2.30 mm to (66.3, 91.8)
- moved C31 2.30 mm to (75.6, 91.9)
- moved C32 2.30 mm to (81.2, 91.2)
- moved C33 2.30 mm to (81.2, 81.7)
- moved C36 2.30 mm to (75.8, 82.1)
- moved C37 2.30 mm to (76.6, 80.5)
- moved D5 2.30 mm to (89.9, 77.0)
- moved D6 2.30 mm to (89.8, 95.4)
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Routing:
- net GND: track 3.16 -> 674.9 mm, vias 0 -> 58
- net +5V_POW: track 0.00 -> 437.7 mm, vias 0 -> 13
- net AREF: track 0.00 -> 289.6 mm, vias 0 -> 22
- net +12V: track 0.00 -> 235.4 mm, vias 0 -> 9
- net MOSI: track 0.00 -> 201.5 mm, vias 0 -> 8
- net RESET: track 0.00 -> 121.8 mm, vias 0 -> 8
- net LED_MOT0: track 0.00 -> 118.0 mm, vias 0 -> 3
- net ADC0: track 0.00 -> 63.0 mm, vias 0 -> 5
- net ADC3: track 0.00 -> 61.0 mm, vias 0 -> 3
- net LED_MOT1: track 0.00 -> 58.9 mm, vias 0 -> 3
- net ADC2: track 0.00 -> 58.4 mm, vias 0 -> 3
- net ADC1: track 0.00 -> 57.7 mm, vias 0 -> 5
- net Quartz_1: track 0.00 -> 56.9 mm, vias 0 -> 1
- net STEP: track 0.00 -> 53.2 mm, vias 0 -> 2
- net Quartz_2: track 0.00 -> 49.0 mm
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- added copper zone on B.Cu, net GND
- added copper zone on F.Cu, net GND
- removed copper zone on In2.Cu, net +12V
- removed copper zone on In2.Cu, net +5V_POW
- removed copper zone on In1.Cu, net GND
Other:
- board size 99 x 97.5 mm -> 99 x 99 mm
- copper layers 4 -> 2
